File: kicad/usb_c_sensor_breakout/MCU.kicad_sch (KiCad schematic)
At the start: 6 parts, among them U3 STM32G031K8Tx

Commit message: Commit 6: Finished PCB + Updated Schematic
Changed lines of the file:
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@@
 	)
 	(hierarchical_label "UART_TX"
-		(shape input)
+		(shape output)
 		(at 134.62 78.74 0)
 		(effects
@@
 	)
 	(hierarchical_label "I2C_SDA"
-		(shape input)
+		(shape bidirectional)
 		(at 83.82 106.68 180)
 		(effects
@@
 	)
 	(hierarchical_label "SWDIO"
-		(shape input)
+		(shape bidirectional)
 		(at 134.62 101.6 0)
 		(effects
@@
 	)
 	(hierarchical_label "SWCLK"
-		(shape input)
+		(shape output)
 		(at 134.62 104.14 0)
 		(effects
@@
 	)
 	(hierarchical_label "I2C_SCL"
-		(shape input)
+		(shape bidirectional)
 		(at 83.82 104.14 180)
 		(effects
